File: HW2+HW3/ME433_PIC32/ME433_PIC32_Schematic.sch (EAGLE design)
At the start: 0 parts

Commit message: Eagle Work
Parts:
- added C1, C2, C3, C4: 0.1uF, ME433_PIC32_Library:C-US025-025X050
- added C5, C6: 10uF, ME433_PIC32_Library:CPOL-USB45181B
- added J1: USB-MB-H, ME433_PIC32_Library:USB-MB-H
- added LED1: Red, led:LED3MM
- added LED2: Green, led:LED3MM
- added R1, R2: 330, ME433_PIC32_Library:R-US_0207/10
- added R3, R4: 10k, ME433_PIC32_Library:R-US_0207/10
- added U$1: PIC32MX250F128B, ME433_PIC32_Library:PIC32MX250F128B
- added U$2: SLIDE, ME433_PIC32_Library:SLIDE
- added U$3: MCP1702, ME433_PIC32_Library:MCP1702
- added U$4: RESET, ME433_PIC32_Library:PB
- added U$5: USER, ME433_PIC32_Library:PB
- added U$6, U$7: CONN_08, ME433_PIC32_Library:CONN_08
- added U$8: PICKIT3, ME433_PIC32_Library:PICKIT3
- added U$9: 8MHz, ME433_PIC32_Library:OSC
Connections:
- new net +3V3: C4.1, C6.+, LED1.A, U$3.3.VOUT
- new net +5V: C3.1, U$2.3, U$3.2.VIN
- new net GND: C1.2, C3.2, C4.2, C6.-, J1.GND, R1.1, R2.1
- new net N$1: J1.VBUS, U$2.2
- new net N$3: LED1.C, R1.2

Commit message: More Eagle Changes
Parts:
- removed U$6, U$7: CONN_08, ME433_PIC32_Library:CONN_08
- added J3, J4: CONN_08, ME433_PIC32_Library:CONN_08
Connections:
- new net A0: J3.8, U$1.2.A0
- new net A1: J3.7, U$1.3.A1
- new net A4/LED: J3.3, LED2.A, U$1.12.A4/LED
- new net B13: J4.6, U$1.24.B13
- new net B14: J4.7, U$1.25.B14
- new net B15: J4.8, U$1.26.B15
- new net B2: J3.6, U$1.6.B2
- new net B3: J3.5, U$1.7.B3
- new net B4/USER: J3.4, R3.2, U$1.11.B4/USER, U$5.1
- new net B7: J4.3, U$1.16.B7
- new net B8: J4.4, U$1.17.B8
- new net B9: J4.5, U$1.18.B9
- new net D+: J1.D+, U$1.21.D+/B10
- new net D-: J1.D-, U$1.22.D-/B11
- new net MCLR: R4.2, U$1.1.MCLR, U$4.1, U$8.1.MCLR
- new net N$2: U$1.9.OSC1/A2, U$9.3.OSC2
- new net N$4: U$1.10.OSC2/A3, U$9.1.OSC1
- new net N$5: C5.+, U$1.20.VCAP
- new net N$6: LED2.C, R2.2
- new net PGC: U$1.5.PGEC1/B1, U$8.5.PGC
- new net PGD: U$1.4.PGED1/B0, U$8.4.PGD
- new net USBID: J1.ID, U$1.14.USBID/B5
- net +3V3: now also C1.1, C2.1, J3.2, R3.1, R4.1, U$1.13.VDD, U$1.23.VUSB3V3, U$1.28.AVDD, U$8.2.VDD
- net +5V: now also J4.2, U$1.15.VBUS
- net GND: now also C2.2, C5.-, J3.1, J4.1, U$1.19.VSS, U$1.27.AVSS, U$1.8.VSS, U$4.2, U$5.2, U$8.3.VSS, U$9.2.GND
Other:
- moved on the sheet: C1, C2, C5, LED2, R2, R3, R4, U$4, U$5, U$8, U$9
