File: HW2+HW3/ME433_PIC32/ME433_PIC32_Schematic.brd (EAGLE design)
At the start: 50 x 50 mm, 22 parts, among them J1 USB-MB-H, J3 CONN_08, J4 CONN_08

Commit message: Created Gerber Files, Ready For Order
Parts:
- moved R1 3.68 mm to (47.5, 43.0), turned to 90 degrees
- moved C4 1.27 mm to (35.8, 45.6)
- moved C6 1.08 mm to (31.6, 45.7)
- moved C3 0.63 mm to (20.6, 41.2), turned to 270 degrees
- moved C1 0.51 mm to (34.3, 36.1)
- moved R2 0.32 mm to (1.46, 9.08), turned to 90 degrees
- moved J4 0.13 mm to (48.8, 16.5)
Connections:
- net GND: now also U$3.1
Routing:
- net +3V3: track 0.00 -> 149.5 mm, vias 0 -> 5
- net +5V: track 0.00 -> 78.5 mm, vias 0 -> 1
- net B4/USER: track 0.00 -> 63.5 mm, vias 0 -> 2
- net MCLR: track 0.00 -> 56.9 mm, vias 0 -> 2
- net USBID: track 0.00 -> 53.0 mm, vias 0 -> 1
- net D+: track 0.00 -> 47.6 mm, vias 0 -> 2
- net D-: track 0.00 -> 46.8 mm, vias 0 -> 2
- net A4/LED: track 0.00 -> 34.7 mm, vias 0 -> 2
- net PGD: track 0.00 -> 32.3 mm
- net PGC: track 0.00 -> 28.4 mm
- net B9: track 0.00 -> 25.6 mm
- net B8: track 0.00 -> 25.6 mm
- net B7: track 0.00 -> 25.6 mm
- net B2: track 0.00 -> 22.4 mm
- net B3: track 0.00 -> 22.1 mm
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- added copper zone on layer 16, net GND
Other:
- board text added: "April 2017"
- board text added: "Greg Niederschulte"
